File: hardware/magnetometer.kicad_pcb (KiCad board)
At the start: 2 copper layers, 29 parts, among them P1 Power, P2 LED, P3 Photodiode, P4 Monitor, P5 Coil, U1 TL071, U2 TL071

Commit message: Board design
Parts:
- added REF***: OSHW-Logo_11.4x12mm_SilkScreen, Symbols:OSHW-Logo_11.4x12mm_SilkScreen, F.Cu at (184.8, 87.6)
- added Ref**: Val**, Board_Outlines:80mmx60mm_holes, F.Cu at (152.4, 101.6)
- JP1: value Coil feedback enable -> Feedback
- JP2: value Lock aquisition enable -> Lock
- moved JP1 72.7 mm to (157.5, 90.8), turned to 270 degrees
- moved U1 71.5 mm to (165.7, 105.4), turned to 90 degrees
- moved R7 68.2 mm to (149.2, 106.7), turned to 90 degrees
- moved RV1 64.7 mm to (153.7, 120.7), turned to 180 degrees
- moved C1 64.5 mm to (188.6, 112.4), turned to 180 degrees
- moved P1 61.8 mm to (167.7, 123.8)
- moved P2 61.0 mm to (175.3, 79.4), turned to 180 degrees
- moved W2 57.3 mm to (170.8, 88.9)
- moved JP2 51.6 mm to (146.1, 90.8), turned to 90 degrees
- moved R4 50.4 mm to (168.3, 110.5), turned to 180 degrees
- moved R1 45.3 mm to (182.9, 106.7), turned to 90 degrees
- moved R9 40.7 mm to (123.8, 96.5), turned to 270 degrees
- moved C2 39.3 mm to (186.6, 118.7)
- moved P5 38.2 mm to (134.5, 79.4), turned to 180 degrees
- moved R10 37.3 mm to (128.9, 88.9), turned to 180 degrees
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Routing:
- net -12VA: track 0.00 -> 134.6 mm, vias 0 -> 1
- net +12VA: track 0.00 -> 124.3 mm
- net Net-(JP1-Pad1): track 0.00 -> 66.4 mm
- net Net-(P3-Pad1): track 0.00 -> 47.2 mm
- net Net-(R6-Pad1): track 0.00 -> 36.1 mm
- net Net-(R10-Pad2): track 0.00 -> 32.8 mm
- net Net-(P2-Pad1): track 0.00 -> 25.1 mm
- net Net-(JP1-Pad2): track 0.00 -> 19.2 mm
- net Net-(R4-Pad1): track 0.00 -> 18.8 mm
- net Net-(P5-Pad1): track 0.00 -> 18.0 mm
- net Net-(R8-Pad2): track 0.00 -> 15.5 mm
- net Net-(JP2-Pad2): track 0.00 -> 5.98 mm
- added copper zone on B.Cu, net GND
- added copper zone on F.Cu, net GND
Other:
- board outline added: 80 x 60 mm
- net class Default: trace_width 0.25 -> 0.5; via_dia 0.6 -> 1.2; via_drill 0.4 -> 0.8
- board text added: "+"
- board text added: "+12V"
- board text added: "-"
- board text added: "-12V"
- board text added: "Coil"
- board text added: "GND"
- board text added: "LED"
- board text added: "Magnetometer board by Sean Leavey and Hugh Potts"
- board text added: "Monitor"
- board text added: "Photodiode"
- board text added: "Power"
- board text added: "S/N"
- board text added: "VERR"
- board text removed: "add serial number area"
